File: sram.kicad_pcb (KiCad board)
At the start: 4 copper layers, 94.6 x 26.3 mm, 25 parts, among them J1 Cache_slot, M1 UM61256AS, M2 UM61256AS, M3 UM61256AS, M4 UM61256AS, M5 UM61256AS, M6 UM61256AS, M7 UM61256AS, M8 UM61256AS, U1 74F244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

Commit message: Final version 2.4
Parts:
- removed CT3: 10uF 16V, Capacitor_Tantalum_SMD:CP_EIA-7132-20_AVX-U
- CB3: moved to F.Cu
- CT1: value 10uF 16V -> 47uF 16V; footprint Capacitor_Tantalum_SMD:CP_EIA-7132-20_AVX-U -> Capacitor_SMD:C_1206_3216Metric_Pad1.33x1.80mm_HandSolder
- CT2: value 10uF 16V -> 47uF 16V; footprint Capacitor_Tantalum_SMD:CP_EIA-7132-20_AVX-U -> Capacitor_SMD:C_1206_3216Metric_Pad1.33x1.80mm_HandSolder; moved to F.Cu
- M1, M2, M3, M4, M5, M6, M7, M8, MD1: value UM61256AS -> IS61C256AL-12JLI; footprint footprints:SOJ28_18P54X7P75_ISI -> footprints:SOIC-28 very wide
- moved CT2 88.3 mm to (212.7, 96.5), turned to -90 degrees
- moved CB3 60.7 mm to (186.4, 82.5), turned to 0 degrees
- moved CB2 22.0 mm to (166.7, 82.5), turned to 180 degrees
- moved CB4 18.6 mm to (212.7, 83.5), turned to -90 degrees
- moved CB1 18.4 mm to (144.1, 83.5)
- moved R2 4.17 mm to (190.9, 82.5)
- moved CT1 2.54 mm to (127.0, 96.5), turned to -90 degrees
- moved R6 2.54 mm to (172.4, 82.5), turned to 0 degrees
- moved M1 2.05 mm to (206.3, 90.8)
- moved M4 1.07 mm to (137.7, 90.8)
- moved R1 0.99 mm to (195.3, 82.5)
- moved M5 0.64 mm to (203.1, 90.8)
- moved M2 0.52 mm to (173.9, 90.8)
- moved J1 0.45 mm to (171.4, 107.5)
- moved R5 0.37 mm to (178.1, 82.5)
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Routing:
- net GND: track 145.5 -> 123.7 mm, vias 37 -> 39
- net +5V: track 77.3 -> 56.6 mm, vias 21 -> 22
- net Bank1_OE: track 147.4 -> 138.5 mm
- net Byte_WE0: track 155.4 -> 148.7 mm
- net CPU_A4: track 53.9 -> 49.0 mm
- net CPU_D3: track 24.1 -> 19.5 mm
- net CPU_D4: track 27.9 -> 23.4 mm
- net CPU_D5: track 27.9 -> 23.9 mm
- net CPU_D6: track 28.9 -> 25.0 mm
- net Bank0_OE: track 161.7 -> 158.3 mm
- net Bank0_CS: track 162.4 -> 159.1 mm
- net CPU_D7: track 30.8 -> 27.5 mm
- net Byte_WE1: track 114.2 -> 111.0 mm
- net Byte_WE3: track 63.1 -> 60.3 mm
- net Cache_A11: track 100.0 -> 97.5 mm
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Other:
- board size 94.6 x 26.3 mm -> 90.8 x 25.9 mm
- board text added: "2.4"
- board text removed: "2.3"
